Commit message: up control

File: zbot_franka_description/urdf/panda.urdf.xacro (robot description, xacro)
@@ -2,6 +2,11 @@
 <robot name="panda" xmlns:xacro="http://www.ros.org/wiki/xacro">
     <link name="world"/>
+    <joint name="world_joint" type="fixed">
+        <parent link="world"/>
+        <child link="base_link"/>
+    </joint>
+    <link name="base_link"/>
     <joint name="fixed" type="fixed">
-      <parent link="world"/>
+      <parent link="base_link"/>
       <child link="panda_link0"/>
     </joint>
@@ -287,36 +292,8 @@
         <dynamics damping="0.3" />
     </joint>
-    <!-- <gazebo reference="panda_link0">
-        <material>Gazebo/Orange</material>
-        <turnGravityOff>true</turnGravityOff>
-    </gazebo>
-    <gazebo reference="panda_link1">
-        <material>Gazebo/Orange</material>
-        <turnGravityOff>true</turnGravityOff>
-    </gazebo>
-    <gazebo reference="panda_link2">
-        <material>Gazebo/Orange</material>
-        <turnGravityOff>true</turnGravityOff>
-    </gazebo>
-    <gazebo reference="panda_link3">
-        <material>Gazebo/Orange</material>
-        <turnGravityOff>true</turnGravityOff>
-    </gazebo>
-    <gazebo reference="panda_link4">
-        <material>Gazebo/Orange</material>
-        <turnGravityOff>true</turnGravityOff>
-    </gazebo>
-    <gazebo reference="panda_link5">
-        <material>Gazebo/Orange</material>
-        <turnGravityOff>true</turnGravityOff>
-    </gazebo>
-    <gazebo reference="panda_link6">
-        <material>Gazebo/Orange</material>
-        <turnGravityOff>true</turnGravityOff>
-    </gazebo> -->
     <!-- ros_control plugin -->
     <gazebo>
         <plugin name="gazebo_ros2_control" filename="libgazebo_ros2_control.so">
-            <parameters>$(find zbot_franka_control)/config/ros2_control_gazebo.yaml</parameters>
+            <parameters>$(find zbot_franka_control)/config/ros2_controllers.yaml</parameters>
         </plugin>
     </gazebo>

Commit message: up urdf

File: zbot_franka_description/urdf/panda.urdf.xacro (robot description, xacro)
@@ -1,5 +1,5 @@
 <?xml version="1.0" ?>
 <robot name="panda" xmlns:xacro="http://www.ros.org/wiki/xacro">
-    <link name="world"/>
+    <!-- <link name="world"/>
     <joint name="world_joint" type="fixed">
         <parent link="world"/>
@@ -10,5 +10,5 @@
       <parent link="base_link"/>
       <child link="panda_link0"/>
-    </joint>
+    </joint> -->
     <link name="panda_link0">
         <visual>
@@ -292,6 +292,5 @@
         <dynamics damping="0.3" />
     </joint>
-    <!-- ros_control plugin -->
-    <gazebo>
+    <!-- <gazebo>
         <plugin name="gazebo_ros2_control" filename="libgazebo_ros2_control.so">
             <parameters>$(find zbot_franka_control)/config/ros2_controllers.yaml</parameters>
@@ -322,4 +321,4 @@
         <xacro:configure_joint joint_name="panda_finger_joint1" initial_position="0.0"/>
         <xacro:configure_joint joint_name="panda_finger_joint2" initial_position="0.0"/>
-    </ros2_control>
+    </ros2_control> -->
 </robot>
